File: KiCad files/Assignment 1/_saved_Assignment 1.sch (KiCad schematic (older format))
At the start: 21 parts, among them Q1 IRLB3034PBF, Q2 IRLB3034PBF, Q3 IRLB3034PBF, Q4 IRLB3034PBF, SW1 SW_Push, SW2 SW_Push, U1 CC56-12EWA

Commit message: Fixed KiCad project file clash issue Added code to ReadMe
Parts:
- Q4: footprint Silicon-Standard:SOT23-3 -> Aesthetics:BREADBOARD_SPACING
Changed lines of the file:
@@
 F 0 "Q4" H 10558 2353 60  0000 L CNN
 F 1 "IRLB3034PBF" H 10558 2247 60  0000 L CNN
-F 2 "Silicon-Standard:SOT23-3" H 10650 2500 60  0001 L CNN
+F 2 "Aesthetics:BREADBOARD_SPACING" H 10650 2500 60  0001 L CNN
 F 3 "https://www.infineon.com/dgdl/irlb3034pbf.pdf?fileId=5546d462533600a40153566027b22585" H 10650 2600 60  0001 L CNN
 F 4 "IRLB3034PBF-ND" H 10650 2700 60  0001 L CNN "Digi-Key_PN"
@@
 	4900 2050 4900 2100
 $Comp
-L power:GND #PWR0101
+L power:GND #PWR01
 U 1 1 5CED5A91
 P 5400 4150
-F 0 "#PWR0101" H 5400 3900 50  0001 C CNN
+F 0 "#PWR01" H 5400 3900 50  0001 C CNN
 F 1 "GND" H 5405 3977 50  0000 C CNN
 F 2 "" H 5400 4150 50  0001 C CNN
